File: audio-mixer/audio-mixer.kicad_pcb (KiCad board)
At the start: 2 copper layers, 50 x 100 mm, 57 parts, among them J1 PJRAS4X2U01X, J2 10118193-0001LF, J3 RCJ-2234, J4 SJ1-3523N, U1 PDME1-S5-D9-S, U2 MC33174, U3 MC33174, U4 MC33174

Commit message: updates schematic and pcb
Parts:
- J1: value PJRAS4X2U01X -> VAL**
Connections:
- J3 pad 1: Net-(J3-Pad1) -> GND
- J3 pad 2: OUTPUT1L -> OUTPUT1R
- J3 pad 3: OUTPUT1R -> OUTPUT1L
- RV1 pad 7: GND -> (no net)
- RV1 pad 8: GND -> (no net)
- RV2 pad 8: GND -> (no net)
Routing:
- net OUTPUT2R: track 36.1 -> 30.0 mm
- net OUTPUT2L: track 21.5 -> 19.0 mm
- removed copper zone on B.Cu, net GND
Other:
- board text added: "github.com/xfbs/audio-mixer"
- board text added: "v1rev1"

Commit message: updates schematic and PCB
Parts:
- J1: value VAL** -> PJRAS4X2U01X
- moved C2 5.89 mm to (115.5, 106.5)
- moved RV4 1.80 mm to (109.0, 72.5)
- moved RV3 1.41 mm to (109.0, 57.0)
- moved RV5 1.41 mm to (109.0, 105.0)
- moved RV2 1.12 mm to (109.0, 41.5)
- moved RV6 1.12 mm to (109.0, 89.5)
- moved RV1 1.00 mm to (109.0, 26.0)
- moved C18 0.50 mm to (103.0, 64.5)
- moved C8 0.50 mm to (103.0, 22.5)
- moved L1 0.50 mm to (112.0, 113.5)
Routing:
- net +12V: track 162.3 -> 0.00 mm, vias 6 -> 0
- net -12V: track 131.4 -> 0.00 mm, vias 6 -> 0
- net MIXEDL: track 88.0 -> 0.00 mm, vias 4 -> 0
- net MIXEDR: track 83.7 -> 0.00 mm, vias 2 -> 0
- net GND: track 67.1 -> 0.00 mm, vias 8 -> 0
- net Net-(RV5-Pad2): track 38.8 -> 0.00 mm, vias 6 -> 0
- net Net-(RV6-Pad2): track 32.2 -> 0.00 mm, vias 6 -> 0
- net Net-(C21-Pad1): track 30.6 -> 0.00 mm
- net Net-(C13-Pad1): track 30.6 -> 0.00 mm
- net OUTPUT2R: track 30.0 -> 0.00 mm, vias 2 -> 0
- net OUTPUT1R: track 29.1 -> 0.00 mm, vias 2 -> 0
- net Net-(C22-Pad1): track 28.3 -> 0.00 mm
- net Net-(C14-Pad1): track 28.1 -> 0.00 mm
- net Net-(RV5-Pad5): track 27.8 -> 0.00 mm, vias 2 -> 0
- net PROC1R: track 24.6 -> 0.00 mm, vias 2 -> 0
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
Commit message: updates design
Parts:
- added R17: 10k, Resistor_SMD:R_0805_2012Metric_Pad1.15x1.40mm_HandSolder, F.Cu at (98.0, 84.0)
- added R18: 10k, Resistor_SMD:R_0805_2012Metric_Pad1.15x1.40mm_HandSolder, F.Cu at (98.0, 87.0)
- added R19: 50k, Resistor_SMD:R_0805_2012Metric_Pad1.15x1.40mm_HandSolder, F.Cu at (102.8, 84.0)
- added R20: 50k, Resistor_SMD:R_0805_2012Metric_Pad1.15x1.40mm_HandSolder, F.Cu at (98.0, 89.9)
- added R21: 10k, Resistor_SMD:R_0805_2012Metric_Pad1.15x1.40mm_HandSolder, F.Cu at (102.8, 87.0)
- added R22: 10k, Resistor_SMD:R_0805_2012Metric_Pad1.15x1.40mm_HandSolder, F.Cu at (107.5, 84.0)
- added R23: 50k, Resistor_SMD:R_0805_2012Metric_Pad1.15x1.40mm_HandSolder, F.Cu at (102.8, 89.9)
- added R24: 50k, Resistor_SMD:R_0805_2012Metric_Pad1.15x1.40mm_HandSolder, F.Cu at (107.5, 87.0)
- moved C3 28.9 mm to (122.0, 114.5), turned to 0 degrees
- moved C4 18.3 mm to (122.0, 107.5), turned to 180 degrees
- moved C23 17.4 mm to (102.0, 103.0), turned to 270 degrees
- moved C2 6.02 mm to (120.0, 102.5), turned to 180 degrees
- moved C26 5.82 mm to (102.0, 91.1)
- moved R10 3.54 mm to (123.0, 39.9)
- moved C18 3.00 mm to (103.0, 67.5)
- moved R13 2.58 mm to (127.0, 39.9)
- moved C17 2.50 mm to (103.0, 73.5)
- moved C16 2.00 mm to (103.0, 52.0)
- moved C7 2.00 mm to (103.0, 27.0)
- moved U4 2.00 mm to (102.0, 97.0), turned to 90 degrees
- moved C6 1.97 mm to (124.5, 32.1)
- moved C5 1.80 mm to (124.5, 50.9)
- moved U3 1.80 mm to (124.5, 57.0)
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Connections:
- RV1 pad 1: Net-(C7-Pad1) -> Net-(C8-Pad1)
- RV1 pad 4: Net-(C8-Pad1) -> Net-(C7-Pad1)
- RV2 pad 1: Net-(C9-Pad1) -> Net-(C10-Pad1)
- RV2 pad 4: Net-(C10-Pad1) -> Net-(C9-Pad1)
- RV3 pad 1: Net-(C15-Pad1) -> Net-(C16-Pad1)
- RV3 pad 4: Net-(C16-Pad1) -> Net-(C15-Pad1)
- RV4 pad 1: Net-(C17-Pad1) -> Net-(C18-Pad1)
- RV4 pad 4: Net-(C18-Pad1) -> Net-(C17-Pad1)
- U2 pad 1: PROC1L -> PROC1R
- U2 pad 13: PROC2R -> PROC2L
- U2 pad 14: PROC2R -> PROC2L
- U2 pad 2: PROC1L -> PROC1R
- U2 pad 6: PROC1R -> PROC1L
- U2 pad 7: PROC1R -> PROC1L
- U2 pad 8: PROC2L -> PROC2R
- U2 pad 9: PROC2L -> PROC2R
- U3 pad 1: PROC3L -> PROC3R
- U3 pad 13: PROC4R -> PROC4L
- U3 pad 14: PROC4R -> PROC4L
- U3 pad 2: PROC3L -> PROC3R
- U3 pad 6: PROC3R -> PROC3L
- U3 pad 7: PROC3R -> PROC3L
- U3 pad 8: PROC4L -> PROC4R
- U3 pad 9: PROC4L -> PROC4R
- U4 pad 1: OUTPUT1L -> OUTPUT2L
- U4 pad 12: Net-(RV6-Pad5) -> Net-(RV5-Pad2)
- U4 pad 13: OUTPUT2R -> Net-(R17-Pad2)
- U4 pad 14: OUTPUT2R -> OUTPUT1L
- U4 pad 2: OUTPUT1L -> Net-(R21-Pad2)
- U4 pad 3: Net-(RV5-Pad2) -> Net-(RV6-Pad2)
- U4 pad 5: Net-(RV6-Pad2) -> Net-(RV6-Pad5)
- U4 pad 6: OUTPUT2L -> Net-(R22-Pad2)
- U4 pad 7: OUTPUT2L -> OUTPUT2R
- U4 pad 9: OUTPUT1R -> Net-(R18-Pad2)
Routing:
- net +12V: track 0.00 -> 112.1 mm, vias 0 -> 2
- net -12V: track 0.00 -> 93.8 mm
- net Net-(C21-Pad1): track 0.00 -> 30.4 mm
- net Net-(C13-Pad1): track 0.00 -> 30.4 mm
- net Net-(C22-Pad1): track 0.00 -> 27.8 mm
- net Net-(C14-Pad1): track 0.00 -> 27.4 mm
- net PROC1L: track 0.00 -> 21.6 mm, vias 0 -> 2
- net GND: track 0.00 -> 21.0 mm
- net PROC2L: track 0.00 -> 20.0 mm, vias 0 -> 2
- net Net-(C19-Pad1): track 0.00 -> 19.4 mm
- net Net-(C11-Pad1): track 0.00 -> 18.4 mm
- net PROC1R: track 0.00 -> 18.1 mm, vias 0 -> 2
- net PROC2R: track 0.00 -> 13.8 mm
- net Net-(C20-Pad1): track 0.00 -> 13.1 mm
- net Net-(C12-Pad1): track 0.00 -> 12.6 mm
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
Commit message: updates schematic and pcb
Parts:
- moved R22 24.9 mm to (98.0, 107.0), turned to 90 degrees
- moved R21 20.2 mm to (105.0, 107.0), turned to 90 degrees
- moved R24 18.7 mm to (98.0, 103.0), turned to 270 degrees
- moved RV5 15.5 mm to (109.0, 89.5)
- moved RV6 15.5 mm to (109.0, 105.0)
- moved C2 13.2 mm to (125.6, 90.6)
- moved R23 12.7 mm to (104.0, 102.5), turned to 180 degrees
- moved C1 10.4 mm to (111.5, 114.0), turned to 180 degrees
- moved R19 8.44 mm to (98.0, 91.0), turned to 90 degrees
- moved R20 7.08 mm to (105.0, 91.0), turned to 90 degrees
- moved R18 7.00 mm to (105.0, 87.0), turned to 270 degrees
- moved C3 6.50 mm to (122.0, 108.0)
- moved R11 5.68 mm to (121.0, 71.0)
- moved R15 5.20 mm to (127.0, 71.1)
- moved R16 5.20 mm to (125.0, 71.1)
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Connections:
- R17 pad 1: Net-(R17-Pad1) -> GND
- R18 pad 1: Net-(R18-Pad1) -> GND
- R19 pad 2: Net-(R17-Pad1) -> Net-(R17-Pad2)
- R20 pad 2: Net-(R18-Pad1) -> Net-(R18-Pad2)
- R21 pad 1: Net-(R21-Pad1) -> GND
- R22 pad 1: Net-(R22-Pad1) -> GND
- R23 pad 2: Net-(R21-Pad1) -> Net-(R21-Pad2)
- R24 pad 2: Net-(R22-Pad1) -> Net-(R22-Pad2)
- U4 pad 1: OUTPUT2L -> OUTPUT2R
- U4 pad 2: Net-(R21-Pad2) -> Net-(R22-Pad2)
- U4 pad 3: Net-(RV6-Pad2) -> Net-(RV6-Pad5)
- U4 pad 5: Net-(RV6-Pad5) -> Net-(RV6-Pad2)
- U4 pad 6: Net-(R22-Pad2) -> Net-(R21-Pad2)
- U4 pad 7: OUTPUT2R -> OUTPUT2L
Routing:
- net MIXEDR: track 2.00 -> 95.6 mm, vias 0 -> 2
- net MIXEDL: track 2.00 -> 89.8 mm, vias 0 -> 4
- net +12V: track 112.1 -> 167.1 mm, vias 2 -> 4
- net -12V: track 93.8 -> 134.1 mm, vias 0 -> 2
- net Net-(C2-Pad1): track 0.00 -> 34.9 mm
- net OUTPUT1R: track 0.00 -> 28.5 mm, vias 0 -> 2
- net OUTPUT2L: track 0.00 -> 25.9 mm, vias 0 -> 2
- net PROC3L: track 0.00 -> 21.4 mm, vias 0 -> 2
- net GND: track 21.0 -> 41.8 mm, vias 0 -> 5
- net VCC: track 0.00 -> 20.5 mm
- net PROC4L: track 0.00 -> 20.2 mm, vias 0 -> 2
- net Net-(RV6-Pad2): track 0.00 -> 18.7 mm
- net PROC3R: track 0.00 -> 18.1 mm, vias 0 -> 2
- net Net-(RV6-Pad5): track 0.00 -> 16.4 mm
- net OUTPUT1L: track 0.00 -> 15.5 mm
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
Commit message: update pcb
Connections:
- RV1 pad 7: (no net) -> GND
- RV1 pad 8: (no net) -> GND
- RV2 pad 7: (no net) -> GND
- RV2 pad 8: (no net) -> GND
- RV3 pad 7: (no net) -> GND
- RV3 pad 8: (no net) -> GND
- RV4 pad 7: (no net) -> GND
- RV4 pad 8: (no net) -> GND
- RV5 pad 7: (no net) -> GND
- RV5 pad 8: (no net) -> GND
- RV6 pad 7: (no net) -> GND
- RV6 pad 8: (no net) -> GND
Routing:
- net GND: track 41.8 -> 105.4 mm, vias 5 -> 10
- added copper zone on B.Cu, net GND

Commit message: updates pcb
Other:
- board text added: "#JLCJLCJLCJLC"
- board text added: "v1-2019-11-13"
- board text removed: "v1rev1"
Changed lines of the file:
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@@
   (general
     (thickness 1.6)
-    (drawings 9)
+    (drawings 10)
     (tracks 450)
     (zones 0)
@@
   (page A4)
   (layers
-    (0 F.Cu signal)
-    (31 B.Cu signal)
+    (0 F.Cu signal hide)
+    (31 B.Cu signal hide)
     (32 B.Adhes user)
     (33 F.Adhes user)
@@
       (padsonsilk false)
       (subtractmaskfromsilk false)
-      (outputformat 4)
+      (outputformat 1)
       (mirror false)
       (drillshape 0)
       (scaleselection 1)
-      (outputdirectory "."))
+      (outputdirectory "../export/v1"))
   )
   (net 0 "")
@@
       (net 1 GND))
   )
+  (gr_text "#JLCJLCJLCJLC" (at 131.5 73.25 270) (layer F.SilkS)
+    (effects (font (size 1 1) (thickness 0.15)))
+  )
   (gr_text github.com/xfbs/audio-mixer (at 131.5 31 270) (layer F.SilkS)
     (effects (font (size 1 1) (thickness 0.15)))
   )
-  (gr_text v1rev1 (at 131.5 66.5 270) (layer B.SilkS)
-    (effects (font (size 1 1) (thickness 0.15)) (justify mirror))
+  (gr_text v1-2019-11-13 (at 131.5 54.5 270) (layer F.SilkS)
+    (effects (font (size 1 1) (thickness 0.15)))
   )
   (gr_text github.com/xfbs/audio-mixer (at 131.5 83 270) (layer B.SilkS)

Commit message: updates pcb
Parts:
- J3: footprint RCJ-2234:RCJ-2221 -> parts:RCJ-2221
Changed lines of the file:
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@@
   (page A4)
   (layers
-    (0 F.Cu signal hide)
-    (31 B.Cu signal hide)
+    (0 F.Cu signal)
+    (31 B.Cu signal)
     (32 B.Adhes user)
     (33 F.Adhes user)
@@
     (mod_text_size 1 1)
     (mod_text_width 0.15)
-    (pad_size 1.4 2.5)
-    (pad_drill 1.2)
+    (pad_size 3.3 2.1)
+    (pad_drill 3.2)
     (pad_to_mask_clearance 0.051)
     (solder_mask_min_width 0.25)
@@
     (add_net VCC)
   )
+  (module parts:RCJ-2221 (layer F.Cu)
+    (at 93 85)
+    (fp_text reference J3 (at -4 -9) (layer F.SilkS)
+      (effects (font (size 1 0.9) (thickness 0.05)))
+    )
+    (fp_text value RCJ-2234 (at -3 10) (layer F.SilkS) hide
+      (effects (font (size 1 0.9) (thickness 0.05)))
+    )
+    (fp_line (start -10.4 5.1) (end -10.4 4.3) (layer F.SilkS) (width 0.25))
+    (fp_line (start -9.252 5.1) (end -10.4 5.1) (layer F.SilkS) (width 0.25))
+    (fp_line (start -10.4 -5.101) (end -10.4 -4.301) (layer F.SilkS) (width 0.25))
+    (fp_line (start -17.05 4.149) (end -10.4 4.149) (layer F.SilkS) (width 0.25))
+    (fp_line (start -17.05 -4.15) (end -17.05 4.149) (layer F.SilkS) (width 0.25))
+    (fp_line (start -10.4 -4.15) (end -17.05 -4.15) (layer F.SilkS) (width 0.25))
+    (fp_line (start -9.25 -7.999) (end -9.25 -5.101) (layer F.SilkS) (width 0.25))
+    (fp_line (start -9.25 12) (end -9.25 5.1) (layer F.SilkS) (width 0.25))
+    (fp_line (start 2.248 12) (end -9.25 12) (layer F.SilkS) (width 0.25))
+    (fp_line (start -3.75 -7.999) (end -9.25 -7.999) (layer F.SilkS) (width 0.25))
+    (fp_line (start -9.252 -5.101) (end -10.4 -5.101) (layer F.SilkS) (width 0.25))
+    (fp_line (start 2.248 -2.699) (end 2.248 12) (layer F.SilkS) (width 0.25))
+    (fp_line (start 2.248 -7.999) (end 2.248 -5.401) (layer F.SilkS) (width 0.25))
+    (fp_line (start 0.25 -7.999) (end 2.25 -7.999) (layer F.SilkS) (width 0.25))
+    (pad 5 thru_hole rect (at -1.75 7.25) (size 3.3 2.1) (drill oval 3.2 2) (layers *.Cu *.Mask)
+      (net 1 GND))
+    (pad 4 thru_hole rect (at -1.75 -7.25) (size 3.3 2.1) (drill oval 3.2 2) (layers *.Cu *.Mask)
+      (net 1 GND))
+    (pad 3 thru_hole circle (at 2.25 -4) (size 1.9 1.9) (drill 1.2) (layers *.Cu *.Mask)
+      (net 18 OUTPUT1L))
+    (pad 2 thru_hole circle (at 1 4) (size 1.9 1.9) (drill 1.2) (layers *.Cu *.Mask)
+      (net 17 OUTPUT1R))
+    (pad 1 thru_hole circle (at -2.25 0) (size 1.9 1.9) (drill 1.2) (layers *.Cu *.Mask)
+      (net 1 GND))
+  )
   (module parts:EVJYK6 (layer B.Cu)
     (at 109 41.5 90)
@@
       (net 8 "Net-(C2-Pad1)"))
   )
-  (module RCJ-2234:RCJ-2221 (layer F.Cu)
-    (at 93 85)
-    (fp_text reference J3 (at -4 -9) (layer F.SilkS)
-      (effects (font (size 1 0.9) (thickness 0.05)))
-    )
-    (fp_text value RCJ-2234 (at -3 10) (layer F.SilkS) hide
-      (effects (font (size 1 0.9) (thickness 0.05)))
-    )
-    (fp_line (start -3.25 -6.4) (end -3.25 -8.1) (layer Edge.Cuts) (width 0.25))
-    (fp_line (start -0.251 -6.4) (end -3.25 -6.4) (layer Edge.Cuts) (width 0.25))
-    (fp_line (start -0.251 -8.1) (end -0.251 -6.4) (layer Edge.Cuts) (width 0.25))
-    (fp_line (start -3.25 -8.1) (end -0.251 -8.1) (layer Edge.Cuts) (width 0.25))
-    (fp_line (start -3.25 6.4) (end -3.25 8.101) (layer Edge.Cuts) (width 0.25))
-    (fp_line (start -0.251 6.4) (end -3.25 6.4) (layer Edge.Cuts) (width 0.25))
-    (fp_line (start -0.251 8.101) (end -0.251 6.4) (layer Edge.Cuts) (width 0.25))
-    (fp_line (start -3.25 8.101) (end -0.251 8.101) (layer Edge.Cuts) (width 0.25))
-    (fp_line (start -10.4 5.1) (end -10.4 4.3) (layer F.SilkS) (width 0.25))
-    (fp_line (start -9.252 5.1) (end -10.4 5.1) (layer F.SilkS) (width 0.25))
-    (fp_line (start -10.4 -5.101) (end -10.4 -4.301) (layer F.SilkS) (width 0.25))
-    (fp_line (start -17.05 4.149) (end -10.4 4.149) (layer F.SilkS) (width 0.25))
-    (fp_line (start -17.05 -4.15) (end -17.05 4.149) (layer F.SilkS) (width 0.25))
-    (fp_line (start -10.4 -4.15) (end -17.05 -4.15) (layer F.SilkS) (width 0.25))
-    (fp_line (start -9.25 -7.999) (end -9.25 -5.101) (layer F.SilkS) (width 0.25))
-    (fp_line (start -9.25 12) (end -9.25 5.1) (layer F.SilkS) (width 0.25))
-    (fp_line (start 2.248 12) (end -9.25 12) (layer F.SilkS) (width 0.25))
-    (fp_line (start -3.75 -7.999) (end -9.25 -7.999) (layer F.SilkS) (width 0.25))
-    (fp_line (start -9.252 -5.101) (end -10.4 -5.101) (layer F.SilkS) (width 0.25))
-    (fp_line (start 2.248 -2.699) (end 2.248 12) (layer F.SilkS) (width 0.25))
-    (fp_line (start 2.248 -7.999) (end 2.248 -5.401) (layer F.SilkS) (width 0.25))
-    (fp_line (start 0.25 -7.999) (end 2.25 -7.999) (layer F.SilkS) (width 0.25))
-    (pad 3 thru_hole circle (at 2.25 -4) (size 1.9 1.9) (drill 1.2) (layers *.Cu *.Mask)
-      (net 18 OUTPUT1L))
-    (pad 2 thru_hole circle (at 1 4) (size 1.9 1.9) (drill 1.2) (layers *.Cu *.Mask)
-      (net 17 OUTPUT1R))
-    (pad 1 thru_hole circle (at -2.25 0) (size 1.9 1.9) (drill 1.2) (layers *.Cu *.Mask)
-      (net 1 GND))
-  )
   (module 10118193-0001LF:FCI_10118193-0001LF (layer F.Cu)

Commit message: updates pcb
Parts:
- added H1: MountingHole, MountingHole:MountingHole_3.2mm_M3, F.Cu at (85.8, 114.2)
- added H2: MountingHole, MountingHole:MountingHole_3.2mm_M3, F.Cu at (130.2, 114.2)
- added H3: MountingHole, MountingHole:MountingHole_3.2mm_M3, F.Cu at (130.2, 19.8)
- added H4: MountingHole, MountingHole:MountingHole_3.2mm_M3, F.Cu at (85.8, 19.8)
- C1, C10, C15, C16, C17, C18, C2, C7, C8, C9: footprint parts:UWJ1E4R7MCL1GB -> Capacitor_SMD:C_Elec_4x5.4
- J4: footprint digikey-footprints:Headphone_Jack_3.5mm_SJ1-3523N -> parts:Headphone_Jack_3.5mm_SJ1-3523N
- moved J1 4.00 mm to (93.0, 51.0)
- moved J4 3.50 mm to (92.0, 104.0)
- moved J3 3.25 mm to (93.0, 88.2)
- turned C10 to 0 degrees
- turned C15 to 0 degrees
- turned C16 to 0 degrees
- turned C17 to 0 degrees
- turned C18 to 0 degrees
- turned C7 to 0 degrees
- turned C8 to 0 degrees
- turned C9 to 0 degrees
Connections:
- C10 pad 1: Net-(C10-Pad1) -> INPUT2R
- C10 pad 2: INPUT2R -> Net-(C10-Pad2)
- C15 pad 1: Net-(C15-Pad1) -> INPUT3L
- C15 pad 2: INPUT3L -> Net-(C15-Pad2)
- C16 pad 1: Net-(C16-Pad1) -> INPUT3R
- C16 pad 2: INPUT3R -> Net-(C16-Pad2)
- C17 pad 1: Net-(C17-Pad1) -> INPUT4L
- C17 pad 2: INPUT4L -> Net-(C17-Pad2)
- C18 pad 1: Net-(C18-Pad1) -> INPUT4R
- C18 pad 2: INPUT4R -> Net-(C18-Pad2)
- C7 pad 1: Net-(C7-Pad1) -> INPUT1L
- C7 pad 2: INPUT1L -> Net-(C7-Pad2)
- C8 pad 1: Net-(C8-Pad1) -> INPUT1R
- C8 pad 2: INPUT1R -> Net-(C8-Pad2)
- C9 pad 1: Net-(C9-Pad1) -> INPUT2L
- C9 pad 2: INPUT2L -> Net-(C9-Pad2)
- J3 pad 4: GND -> (no net)
- J3 pad 5: GND -> (no net)
- RV1 pad 1: Net-(C8-Pad1) -> Net-(C8-Pad2)
- RV1 pad 4: Net-(C7-Pad1) -> Net-(C7-Pad2)
- RV2 pad 1: Net-(C10-Pad1) -> Net-(C10-Pad2)
- RV2 pad 4: Net-(C9-Pad1) -> Net-(C9-Pad2)
- RV3 pad 1: Net-(C16-Pad1) -> Net-(C16-Pad2)
- RV3 pad 4: Net-(C15-Pad1) -> Net-(C15-Pad2)
- RV4 pad 1: Net-(C18-Pad1) -> Net-(C18-Pad2)
- RV4 pad 4: Net-(C17-Pad1) -> Net-(C17-Pad2)
Routing:
- net Net-(C9-Pad2): track 0.00 -> 4.20 mm
- net Net-(C9-Pad1): track 4.20 -> 0.00 mm
- net Net-(C8-Pad2): track 0.00 -> 4.20 mm
- net Net-(C8-Pad1): track 4.20 -> 0.00 mm
- net Net-(C7-Pad2): track 0.00 -> 4.20 mm
- net Net-(C7-Pad1): track 4.20 -> 0.00 mm
- net Net-(C18-Pad2): track 0.00 -> 4.20 mm
- net Net-(C18-Pad1): track 4.20 -> 0.00 mm
- net Net-(C17-Pad2): track 0.00 -> 4.20 mm
- net Net-(C17-Pad1): track 4.20 -> 0.00 mm
- net Net-(C16-Pad2): track 0.00 -> 4.20 mm
- net Net-(C16-Pad1): track 4.20 -> 0.00 mm
- net Net-(C15-Pad2): track 0.00 -> 4.20 mm
- net Net-(C15-Pad1): track 4.20 -> 0.00 mm
- net Net-(C10-Pad2): track 0.00 -> 4.20 mm
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