File: audio-mixer/audio-mixer.kicad_pcb (KiCad board)
At the start: 2 copper layers, 50 x 100 mm, 69 parts, among them J1 PJRAS4X2U01X, J2 10118193-0001LF, J3 RCJ-2234, J4 SJ1-3523N, U1 PDME1-S5-D9-S, U2 MC33174, U3 MC33174, U4 MC33174

Commit message: updates pcb
Parts:
- moved U1 6.00 mm to (129.5, 92.0)
- moved C2 4.35 mm to (125.8, 86.2)
- moved J2 2.06 mm to (100.5, 115.5)
Changed lines of the file:
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@@
   )
   (module Capacitor_SMD:C_Elec_4x5.4 (layer F.Cu)
-    (at 125.5966 90.6 180)
+    (at 125.75 86.25 180)
     (descr "SMD capacitor, aluminum electrolytic nonpolar, 4.0x5.4mm")
     (tags "capacitor electrolyic nonpolar")
@@
   )
   (module PDME1-S5-D9-S:CONV_PDME1-S5-D9-S (layer F.Cu)
-    (at 129.5 98 270)
+    (at 129.5 92 270)
     (fp_text reference U1 (at -4 0.5 180) (layer F.SilkS)
       (effects (font (size 1 1) (thickness 0.05)))
@@
   )
   (module 10118193-0001LF:FCI_10118193-0001LF (layer F.Cu)
-    (at 102.5 115)
+    (at 100.5 115.5)
     (attr smd)
     (fp_text reference J2 (at 0 -4.48892) (layer F.SilkS)
